File: fleet_tracker.kicad_pcb (KiCad board)
At the start: 2 copper layers, 80 x 70 mm, 21 parts, among them J1 DB128V-5.08-5P-GN-S, J2 2685Y-116CNG1SNA01, J3 2685Y-116CNG1SNA01, U2 TJA1051T/3/1J, U3 TSR 1-2450E

Commit message: generate bom files
Routing:
- net /+24V_FUSED: track 19.9 -> 19.4 mm
Other:
- board text removed: "Designed by B Amorim"
- board text removed: "XCOPE AI"
Changed lines of the file:
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@@
 		(allow_soldermask_bridges_in_footprints no)
 		(tenting front back)
+		(aux_axis_origin 104.5 150.5)
 		(grid_origin 105 70)
 		(pcbplotparams
@@
 			(drillshape 0)
 			(scaleselection 1)
-			(outputdirectory "")
+			(outputdirectory "gerbers/")
 		)
 	)
@@
 		)
 		(pad "2" thru_hole oval
-			(at 11 0)
+			(at 11.5 0)
 			(size 1 2.2)
 			(drill oval 0.599998 1.699997)
@@
 	)
 	(gr_text "IGN"
-		(at 107 129.16 90)
+		(at 106 129.16 270)
 		(layer "F.SilkS")
 		(effects
@@
 	)
 	(gr_text "CAN_L"
-		(at 107 119 90)
+		(at 106 119 270)
 		(layer "F.SilkS")
 		(effects
@@
 	)
 	(gr_text "CAN_H"
-		(at 107 124.08 90)
+		(at 106 124.08 270)
 		(layer "F.SilkS")
 		(effects
@@
 	)
 	(gr_text "GND"
-		(at 107 113.92 90)
+		(at 106 113.92 270)
 		(layer "F.SilkS")
 		(effects
@@
 	)
 	(gr_text "+24V"
-		(at 107 134.24 90)
+		(at 106 134.24 270)
 		(layer "F.SilkS")
 		(effects
@@
 		)
 	)
-	(gr_text "XCOPE AI"
-		(at 109.5 109 90)
-		(layer "F.SilkS")
-		(effects
-			(font
-				(size 1.5 1.5)
-				(thickness 0.3)
-				(bold yes)
-			)
-			(justify left bottom)
-		)
-	)
-	(gr_text "Designed by B Amorim"
-		(at 111.5 109 90)
-		(layer "F.SilkS")
-		(effects
-			(font
-				(size 1 1)
-				(thickness 0.2)
-				(bold yes)
-			)
-			(justify left bottom)
-		)
-	)
 	(segment
 		(start 141.31 108.69)
@@
 	)
 	(segment
-		(start 152 141.5)
-		(end 155 138.5)
+		(start 145.5 140.5)
+		(end 151 140.5)
 		(width 0.5)
 		(layer "F.Cu")
@@
 	)
 	(segment
-		(start 145 140.5)
-		(end 151 140.5)
+		(start 152 141.5)
+		(end 155 138.5)
 		(width 0.5)
 		(layer "F.Cu")
@@
 		(name "$teardrop_padvia$")
 		(hatch none 0.1)
-		(priority 30006)
+		(priority 30011)
 		(attr
 			(teardrop
@@
 		(polygon
 			(pts
-				(xy 162.594236 144.25) (xy 162.594236 143.75) (xy 162.058527 143.705764) (xy 161.999 144) (xy 162.058527 144.294236)
+				(xy 121.553749 122.405764) (xy 121.053749 122.405764) (xy 121.009513 122.941473) (xy 121.303749 123.001)
+				(xy 121.597985 122.941473)
 			)
 		)
@@
 		(name "$teardrop_padvia$")
 		(hatch none 0.1)
-		(priority 30007)
+		(priority 30010)
 		(attr
 			(teardrop
@@
 		(name "$teardrop_padvia$")
 		(hatch none 0.1)
-		(priority 30008)
+		(priority 30000)
 		(attr
 			(teardrop
@@
 		(name "$teardrop_padvia$")
 		(hatch none 0.1)
-		(priority 30003)
+		(priority 30002)
 		(attr
 			(teardrop
@@
 		(polygon
 			(pts
-				(xy 152.25 148.405764) (xy 151.75 148.405764) (xy 151.705764 148.941473) (xy 152 149.001) (xy 152.294236 148.941473)
+				(xy 126.75 131.405764) (xy 126.25 131.405764) (xy 126.205764 131.941473) (xy 126.5 132.001) (xy 126.794236 131.941473)
 			)
 		)
@@
 		(name "$teardrop_padvia$")
 		(hatch none 0.1)
-		(priority 30001)
+		(priority 30013)
 		(attr
 			(teardrop
@@
 		(polygon
 			(pts
-				(xy 133.25 133.905764) (xy 132.75 133.905764) (xy 132.705764 134.441473) (xy 133 134.501) (xy 133.294236 134.441473)
+				(xy 144.379037 120.171736) (xy 144.025485 120.525288) (xy 144.059513 120.938527) (xy 144.354456 120.880707)
+				(xy 144.647985 120.821473)
 			)
 		)
@@
 		(name "$teardrop_padvia$")
 		(hatch none 0.1)
-		(priority 30011)
+		(priority 30009)
 		(attr
 			(teardrop
@@
 		(polygon
 			(pts
-				(xy 132.67 108.905764) (xy 132.17 108.905764) (xy 132.125764 109.441473) (xy 132.42 109.501) (xy 132.714236 109.441473)
+				(xy 152.25 148.405764) (xy 151.75 148.405764) (xy 151.705764 148.941473) (xy 152 149.001) (xy 152.294236 148.941473)
 			)
 		)
@@
 		(name "$teardrop_padvia$")
 		(hatch none 0.1)
-		(priority 30004)
+		(priority 30003)
 		(attr
 			(teardrop
@@
 		(polygon
 			(pts
-				(xy 131.103749 114.094236) (xy 131.603749 114.094236) (xy 131.647985 113.558527) (xy 131.353749 113.499)
-				(xy 131.059513 113.558527)
+				(xy 162.594236 144.25) (xy 162.594236 143.75) (xy 162.058527 143.705764) (xy 161.999 144) (xy 162.058527 144.294236)
 			)
 		)
@@
 		(name "$teardrop_padvia$")
 		(hatch none 0.1)
-		(priority 30002)
+		(priority 30007)
 		(attr
 			(teardrop
@@
 		(polygon
 			(pts
-				(xy 118.405764 113.67) (xy 118.405764 114.17) (xy 118.941473 114.214236) (xy 119.001 113.92) (xy 118.941473 113.625764)
+				(xy 161.405764 143.75) (xy 161.405764 144.25) (xy 161.941473 144.294236) (xy 162.001 144) (xy 161.941473 143.705764)
 			)
 		)
@@
 		(name "$teardrop_padvia$")
 		(hatch none 0.1)
-		(priority 30012)
+		(priority 30008)
 		(attr
 			(teardrop
@@
 		(polygon
 			(pts
-				(xy 132.67 89.405764) (xy 132.17 89.405764) (xy 132.125764 89.941473) (xy 132.42 90.001) (xy 132.714236 89.941473)
+				(xy 131.103749 114.094236) (xy 131.603749 114.094236) (xy 131.647985 113.558527) (xy 131.353749 113.499)
+				(xy 131.059513 113.558527)
 			)
 		)
@@
 		(name "$teardrop_padvia$")
 		(hatch none 0.1)
-		(priority 30005)
+		(priority 30012)
 		(attr
 			(teardrop
@@
 		(polygon
 			(pts
-				(xy 161.405764 143.75) (xy 161.405764 144.25) (xy 161.941473 144.294236) (xy 162.001 144) (xy 161.941473 143.705764)
+				(xy 132.67 89.405764) (xy 132.17 89.405764) (xy 132.125764 89.941473) (xy 132.42 90.001) (xy 132.714236 89.941473)
 			)
 		)
@@
 		(name "$teardrop_padvia$")
 		(hatch none 0.1)
-		(priority 30013)
+		(priority 30001)
 		(attr
 			(teardrop
@@
 		(polygon
 			(pts
-				(xy 144.379037 120.171736) (xy 144.025485 120.525288) (xy 144.059513 120.938527) (xy 144.354456 120.880707)
-				(xy 144.647985 120.821473)
+				(xy 165.69 109.405764) (xy 165.19 109.405764) (xy 165.145764 109.941473) (xy 165.44 110.001) (xy 165.734236 109.941473)
 			)
 		)
@@
 		(name "$teardrop_padvia$")
 		(hatch none 0.1)
-		(priority 30000)
+		(priority 30006)
 		(attr
 			(teardrop
@@
 		(polygon
 			(pts
-				(xy 126.75 131.405764) (xy 126.25 131.405764) (xy 126.205764 131.941473) (xy 126.5 132.001) (xy 126.794236 131.941473)
+				(xy 118.405764 113.67) (xy 118.405764 114.17) (xy 118.941473 114.214236) (xy 119.001 113.92) (xy 118.941473 113.625764)
 			)
 		)
@@
 		(name "$teardrop_padvia$")
 		(hatch none 0.1)
-		(priority 30009)
+		(priority 30005)
 		(attr
 			(teardrop
@@
 		(polygon
 			(pts
-				(xy 121.553749 122.405764) (xy 121.053749 122.405764) (xy 121.009513 122.941473) (xy 121.303749 123.001)
-				(xy 121.597985 122.941473)
+				(xy 132.67 108.905764) (xy 132.17 108.905764) (xy 132.125764 109.441473) (xy 132.42 109.501) (xy 132.714236 109.441473)
 			)
 		)
@@
 		(net_name "GND")
 		(layer "F.Cu")
-		(hatch edge 0.5)
-		(connect_pads
-			(clearance 0.5)
+		(name "$teardrop_padvia$")
+		(hatch none 0.1)
+		(priority 30004)
+		(attr
+			(teardrop
+				(type padvia)
+			)
 		)
-		(min_thickness 0.25)
+		(connect_pads yes
+			(clearance 0)
+		)
+		(min_thickness 0.0254)
 		(filled_areas_thickness no)
 		(fill yes
 			(thermal_gap 0.5)
 			(thermal_bridge_width 0.5)
+			(island_removal_mode 1)
+			(island_area_min 10)
 		)
 		(polygon
 			(pts
-				(xy 185 80) (xy 105 80) (xy 105 150) (xy 185 150)
+				(xy 133.25 133.905764) (xy 132.75 133.905764) (xy 132.705764 134.441473) (xy 133 134.501) (xy 133.294236 134.441473)
 			)
 		)
@@
 		(net_name "GND")
 		(layer "F.Cu")
-		(name "$teardrop_padvia$")
-		(hatch none 0.1)
-		(priority 30010)
-		(attr
-			(teardrop
-				(type padvia)
-			)
-		)
-		(connect_pads yes
-			(clearance 0)
+		(hatch edge 0.5)
+		(connect_pads
+			(clearance 0.5)
 		)
-		(min_thickness 0.0254)
+		(min_thickness 0.25)
 		(filled_areas_thickness no)
 		(fill yes
 			(thermal_gap 0.5)
 			(thermal_bridge_width 0.5)
-			(island_removal_mode 1)
-			(island_area_min 10)
 		)
 		(polygon
 			(pts
-				(xy 165.69 109.405764) (xy 165.19 109.405764) (xy 165.145764 109.941473) (xy 165.44 110.001) (xy 165.734236 109.941473)
+				(xy 185 80) (xy 105 80) (xy 105 150) (xy 185 150)
 			)
 		)

Commit message: final changes before review
Parts:
- C1: renamed from C2; value CL10B104KB8NNNC -> 100nF 50V X7R
- C2: renamed from C1; value CL10B104KB8NNNC -> 100nF 50V X7R
- C3, C4: value CL31B106KBHNNNE -> 10uF 50V X7R
- D1: value SMBJ33CA-C78420 -> SMBJ33CA 33V
- D2: value SMAJ5.0CA_C10756 -> SMAJ5.0CA 5V
- D3: value NUP2105LT1G -> NUP2105LT1G 24V
- F1: value 5x20 BLX-Atype Fuse holder XC-7 -> 5x20 Fuse holder 1 A fast-blow
- J1: value DB128V-5.08-5P-GN-S -> Truck Side FMS
- J2, J3: value 2685Y-116CNG1SNA01 -> 1×16 2.54 mm socket
- L1: value ACT45B-101-2P-TL003 -> 100µH
- R1: value HOAR0603-1/10W-100KR-1%-TCR25 -> 100k
- R2: value RC0603FR-0710KL -> 10k
- U1: renamed from U2; value TJA1051T/3/1J -> TJA1051
- moved C1 11.1 mm to (131.4, 115.5), turned to 90 degrees
- moved C2 10.5 mm to (141.1, 119.6), turned to 0 degrees
- moved H1 1.00 mm to (109.0, 85.0)
- moved H2 1.00 mm to (179.0, 85.0)
- moved H3 1.00 mm to (109.0, 145.0)
- moved H4 1.00 mm to (179.0, 145.0)
- renumbered REF** to H1, REF** to H2, REF** to H3, REF** to H4, U3 to U2
Connections:
- C1 pad 1: /+5V -> +3.3V
- C2 pad 1: +3.3V -> /+5V
Routing:
- net +3.3V: track 54.8 -> 53.8 mm
- net /+5V: track 91.6 -> 91.0 mm
- net GND: track 52.4 -> 52.9 mm
Other:
- board text added: "1A fast-blow"
- board text added: "2.54mm"
- board text added: "24VDC (9-32V)"
- board text added: "5.08mm"
- board text added: "FleetTrackerV0 07/2026"
- board text added: "LilyGo T-SIM7080G-S3"
- board text removed: "FleetTrackerV0"
